File: hardware/pcb/receiver/receiver.brd (EAGLE design)
At the start: 100 x 100 mm, 82 parts, among them X1 5-1634506-1H

Commit message: hw: board misc changes
Parts:
- H5, H6: device holes:3,3 -> holes:3,3@1
- R10: device rcl:M0805 -> rcl:R0805
- moved C37 0.76 mm to (39.6, 48.0)
- moved L1 0.25 mm to (32.6, 25.7)
- moved L2 0.25 mm to (32.5, 32.3)
- moved L3 0.25 mm to (32.5, 38.9)
Routing:
- net N$15: track 1.65 -> 2.42 mm
- net +3V3A_ADC: track 57.2 -> 58.0 mm
- net N$18: track 10.5 -> 11.0 mm
- net N$17: track 10.5 -> 11.0 mm
- net GND: vias 362 -> 364

Commit message: hw: board final touches
Parts:
- added J3, J4: (no value), con-amp:10X02MTA
- moved C39 0.94 mm to (59.3, 81.6), turned to 0 degrees
- moved C33 0.25 mm to (62.2, 48.0)
- moved C22 0.25 mm to (63.8, 52.5)
Connections:
- net +3V3: now also J4.2
- net +5V: now also J3.2
- net GND: now also J3.1, J4.1
Routing:
- net +5V: track 52.1 -> 57.9 mm
- net +3V3: track 52.7 -> 55.7 mm
- net GND: track 80.9 -> 78.2 mm, vias 364 -> 375
- net N$19: track 1.36 -> 2.49 mm
- net VCM: track 24.5 -> 25.2 mm

Commit message: hw: final changes
Parts:
- moved H6 7.50 mm to (6.00, 28.0)
- moved X1 5.72 mm to (17.0, 40.0)
- moved H5 3.06 mm to (27.0, 52.0)
Routing:
- net N$2: track 55.9 -> 55.0 mm
Changed lines of the file:
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@@
 <setting verticaltext="up"/>
 </settings>
-<grid distance="10" unitdist="mil" unit="mm" style="lines" multiple="1" display="yes" altdistance="1" altunitdist="mil" altunit="mil"/>
+<grid distance="10" unitdist="mil" unit="mm" style="lines" multiple="1" display="yes" altdistance="5" altunitdist="mil" altunit="mil"/>
 <layers>
 <layer number="1" name="Top" color="4" fill="1" visible="yes" active="yes"/>
@@
 <element name="C2" library="rcl" package="C0805" value="100n" x="69.85" y="69.469" smashed="yes" rot="R270">
 <attribute name="MFR" value="C0805C104K5RACTU" x="69.85" y="69.469" size="1.778" layer="27" rot="R270" display="off"/>
-<attribute name="NAME" x="68.834" y="73.787" size="1.27" layer="25" rot="R270"/>
+<attribute name="NAME" x="69.088" y="73.787" size="1.27" layer="25" rot="R270"/>
 <attribute name="VALUE" x="67.31" y="70.739" size="1.27" layer="27" rot="R270"/>
 </element>
@@
 <attribute name="NAME" x="81.915" y="18.923" size="1.27" layer="25" ratio="10"/>
 </element>
-<element name="X1" library="lstolcman_thesis" package="5-1634506-1" value="5-1634506-1H" x="17.018" y="45.72" smashed="yes" rot="R90">
-<attribute name="MFR" value="5-1634506-1" x="17.018" y="45.72" size="1.778" layer="27" rot="R90" display="off"/>
-<attribute name="NAME" x="17.98" y="53.24" size="1.27" layer="25" rot="R180"/>
-<attribute name="VALUE" x="24.738" y="42.98" size="1.27" layer="27" rot="R90"/>
+<element name="X1" library="lstolcman_thesis" package="5-1634506-1" value="5-1634506-1H" x="17.018" y="40" smashed="yes" rot="R90">
+<attribute name="MFR" value="5-1634506-1" x="17.018" y="40" size="1.778" layer="27" rot="R90" display="off"/>
+<attribute name="NAME" x="17.98" y="47.52" size="1.27" layer="25" rot="R180"/>
+<attribute name="VALUE" x="24.738" y="37.26" size="1.27" layer="27" rot="R90"/>
 </element>
 <element name="H1" library="holes" package="3,3" value="MOUNT-HOLE3.3" x="4" y="4"/>
@@
 <attribute name="VALUE" x="12.8189" y="83.3181" size="1.27" layer="27" rot="R270"/>
 </element>
-<element name="H5" library="holes" package="3,3@1" value="MOUNT-HOLE3.3" x="28.32" y="54.764"/>
-<element name="H6" library="holes" package="3,3@1" value="MOUNT-HOLE3.3" x="6.73" y="35.46"/>
+<element name="H5" library="holes" package="3,3@1" value="MOUNT-HOLE3.3" x="27" y="52"/>
+<element name="H6" library="holes" package="3,3@1" value="MOUNT-HOLE3.3" x="6" y="28"/>
 <element name="J3" library="con-amp" package="10X02MTA" value="" x="48.514" y="93.218">
 <attribute name="MFR" value="640454-2" x="48.514" y="93.218" size="1.778" layer="27" display="off"/>
@@
 <vertex x="75.946" y="101.6"/>
 <vertex x="75.946" y="68.072"/>
-<vertex x="72.39" y="63.5"/>
-<vertex x="72.39" y="51.816"/>
-<vertex x="71.501" y="51.816"/>
-<vertex x="71.501" y="73.406"/>
-<vertex x="59.436" y="73.406"/>
-<vertex x="58.928" y="73.914"/>
-<vertex x="58.928" y="75.692"/>
-<vertex x="59.436" y="76.2"/>
-<vertex x="71.628" y="76.2"/>
+<vertex x="72.136" y="63.5"/>
+<vertex x="72.136" y="52.324"/>
+<vertex x="71.628" y="52.324"/>
+<vertex x="71.628" y="72.136"/>
+<vertex x="57.15" y="72.136"/>
+<vertex x="56.642" y="72.644"/>
+<vertex x="56.642" y="74.422"/>
+<vertex x="57.15" y="74.93"/>
+<vertex x="71.628" y="74.93"/>
 <vertex x="71.628" y="100.33"/>
 </polygon>
@@
 <vertex x="75.946" y="102.362"/>
 <vertex x="75.946" y="68.072"/>
-<vertex x="72.39" y="63.5"/>
-<vertex x="72.39" y="51.816"/>
-<vertex x="71.501" y="51.816"/>
-<vertex x="71.501" y="73.406"/>
-<vertex x="59.436" y="73.406"/>
-<vertex x="58.928" y="73.914"/>
-<vertex x="58.928" y="75.692"/>
-<vertex x="59.436" y="76.2"/>
-<vertex x="71.628" y="76.2"/>
+<vertex x="72.136" y="63.246"/>
+<vertex x="72.136" y="52.324"/>
+<vertex x="71.501" y="52.324"/>
+<vertex x="71.628" y="72.136"/>
+<vertex x="57.15" y="72.136"/>
+<vertex x="56.642" y="72.644"/>
+<vertex x="56.642" y="74.422"/>
+<vertex x="57.15" y="74.93"/>
+<vertex x="71.628" y="74.93"/>
 <vertex x="71.628" y="100.33"/>
 </polygon>
@@
 <via x="53.848" y="80.518" extent="1-16" drill="0.4" diameter="0.6"/>
 <via x="56.1594" y="77.3938" extent="1-16" drill="0.4" diameter="0.6"/>
-<via x="56.642" y="74.422" extent="1-16" drill="0.4" diameter="0.6"/>
-<via x="52.324" y="78.486" extent="1-16" drill="0.4" diameter="0.6"/>
+<via x="55.88" y="74.93" extent="1-16" drill="0.4" diameter="0.6"/>
+<via x="50.8" y="78.486" extent="1-16" drill="0.4" diameter="0.6"/>
 <via x="61.468" y="84.582" extent="1-16" drill="0.4" diameter="0.6"/>
 <via x="61.468" y="88.646" extent="1-16" drill="0.4" diameter="0.6"/>
 <via x="61.468" y="86.614" extent="1-16" drill="0.4" diameter="0.6"/>
-<via x="70.358" y="78.232" extent="1-16" drill="0.4" diameter="0.6"/>
-<via x="66.294" y="79.502" extent="1-16" drill="0.4" diameter="0.6"/>
+<via x="69.088" y="76.708" extent="1-16" drill="0.4" diameter="0.6"/>
+<via x="66.548" y="78.74" extent="1-16" drill="0.4" diameter="0.6"/>
 <via x="68.834" y="86.868" extent="1-16" drill="0.4" diameter="0.6" alwaysstop="yes"/>
 <via x="69.596" y="82.296" extent="1-16" drill="0.4" diameter="0.6"/>
@@
 <via x="49.276" y="85.09" extent="1-16" drill="0.4" diameter="0.6"/>
 <via x="50.292" y="81.28" extent="1-16" drill="0.4" diameter="0.6"/>
-<via x="50.038" y="77.978" extent="1-16" drill="0.4" diameter="0.6"/>
-<via x="52.324" y="75.692" extent="1-16" drill="0.4" diameter="0.6"/>
+<via x="52.07" y="76.708" extent="1-16" drill="0.4" diameter="0.6"/>
+<via x="50.546" y="74.168" extent="1-16" drill="0.4" diameter="0.6"/>
 <via x="52.324" y="72.39" extent="1-16" drill="0.4" diameter="0.6"/>
 <via x="50.038" y="70.358" extent="1-16" drill="0.4" diameter="0.6"/>
@@
 <via x="61.214" y="67.056" extent="1-16" drill="0.4" diameter="0.6"/>
 <via x="57.404" y="64.008" extent="1-16" drill="0.4" diameter="0.6"/>
-<via x="67.564" y="70.612" extent="1-16" drill="0.4" diameter="0.6"/>
-<via x="70.612" y="72.644" extent="1-16" drill="0.4" diameter="0.6"/>
-<via x="64.77" y="70.612" extent="1-16" drill="0.4" diameter="0.6"/>
-<via x="60.706" y="70.866" extent="1-16" drill="0.4" diameter="0.6"/>
+<via x="67.564" y="70.866" extent="1-16" drill="0.4" diameter="0.6"/>
+<via x="65.024" y="71.12" extent="1-16" drill="0.4" diameter="0.6"/>
+<via x="61.976" y="70.612" extent="1-16" drill="0.4" diameter="0.6"/>
+<via x="59.182" y="70.866" extent="1-16" drill="0.4" diameter="0.6"/>
 <via x="56.642" y="71.12" extent="1-16" drill="0.4" diameter="0.6"/>
-<via x="59.5122" y="76.581" extent="1-16" drill="0.4" diameter="0.6"/>
+<via x="63.5762" y="76.581" extent="1-16" drill="0.4" diameter="0.6"/>
 <via x="84.074" y="29.21" extent="1-16" drill="0.4" diameter="0.6"/>
 <via x="84.836" y="19.05" extent="1-16" drill="0.4" diameter="0.6"/>
@@
 <via x="39.37" y="58.674" extent="1-16" drill="0.4" diameter="0.6"/>
 <via x="10.668" y="58.674" extent="1-16" drill="0.4" diameter="0.6"/>
-<via x="34.29" y="58.42" extent="1-16" drill="0.4" diameter="0.6"/>
+<via x="34.036" y="55.88" extent="1-16" drill="0.4" diameter="0.6"/>
 <via x="22.098" y="58.674" extent="1-16" drill="0.4" diameter="0.6"/>
 <via x="16.256" y="58.674" extent="1-16" drill="0.4" diameter="0.6"/>
 <via x="4.826" y="58.674" extent="1-16" drill="0.4" diameter="0.6"/>
-<via x="25.654" y="48.768" extent="1-16" drill="0.4" diameter="0.6"/>
+<via x="30.226" y="58.166" extent="1-16" drill="0.4" diameter="0.6"/>
 <via x="30.988" y="47.498" extent="1-16" drill="0.4" diameter="0.6"/>
-<via x="36.322" y="54.61" extent="1-16" drill="0.4" diameter="0.6"/>
+<via x="38.354" y="55.118" extent="1-16" drill="0.4" diameter="0.6"/>
 <via x="11.684" y="45.72" extent="1-16" drill="0.4" diameter="0.6"/>
 <via x="17.018" y="50.292" extent="1-16" drill="0.4" diameter="0.6"/>
@@
 <via x="59.436" y="21.59" extent="1-16" drill="0.4" diameter="0.6"/>
 <via x="55.372" y="93.726" extent="1-16" drill="0.4" diameter="0.6" alwaysstop="yes"/>
-<via x="78.74" y="76.962" extent="1-16" drill="0.4" diameter="0.6" alwaysstop="yes"/>
+<via x="77.978" y="76.962" extent="1-16" drill="0.4" diameter="0.6" alwaysstop="yes"/>
 <via x="84.074" y="74.93" extent="1-16" drill="0.4" diameter="0.6" alwaysstop="yes"/>
 <via x="94.742" y="85.344" extent="1-16" drill="0.4" diameter="0.6"/>
@@
 <via x="9.398" y="23.622" extent="1-16" drill="0.4" diameter="0.6"/>
 <via x="10.922" y="29.21" extent="1-16" drill="0.4" diameter="0.6"/>
-<via x="4.318" y="26.924" extent="1-16" drill="0.4" diameter="0.6"/>
+<via x="4.826" y="36.83" extent="1-16" drill="0.4" diameter="0.6"/>
 <via x="5.842" y="18.542" extent="1-16" drill="0.4" diameter="0.6"/>
 <via x="10.414" y="13.716" extent="1-16" drill="0.4" diameter="0.6"/>
@@
 <via x="45.466" y="91.186" extent="1-16" drill="0.4" diameter="0.6"/>
 <via x="44.958" y="93.98" extent="1-16" drill="0.4" diameter="0.6"/>
+<wire x1="20.448" y1="36.57" x2="19.304" y2="37.592" width="0" layer="19" extent="1-1"/>
+<wire x1="14.732" y1="35.306" x2="13.588" y2="36.57" width="0" layer="19" extent="1-1"/>
 </signal>
 <signal name="N$2">
@@
 <contactref element="R10" pad="2"/>
 <contactref element="X1" pad="1"/>
-<wire x1="17.079" y1="45.273" x2="17.018" y2="45.72" width="0.6096" layer="1"/>
+<wire x1="17.079" y1="45.273" x2="17.018" y2="40" width="0.6096" layer="1"/>
 <wire x1="35.56" y1="18.1" x2="35.56" y2="16.764" width="0.6096" layer="1"/>
 <wire x1="35.56" y1="16.764" x2="34.29" y2="15.494" width="0.6096" layer="1"/>
@@
 <wire x1="22.86" y1="15.494" x2="18.288" y2="15.494" width="0.6096" layer="1"/>
 <wire x1="18.288" y1="15.494" x2="17.018" y2="16.764" width="0.6096" layer="1"/>
-<wire x1="17.018" y1="16.764" x2="17.018" y2="45.72" width="0.6096" layer="1"/>
+<wire x1="17.018" y1="16.764" x2="17.018" y2="40" width="0.6096" layer="1"/>
 <wire x1="22.733" y1="15.56" x2="22.86" y2="15.56" width="0.3048" layer="1"/>
 <wire x1="22.86" y1="15.56" x2="22.86" y2="15.494" width="0.3048" layer="1"/>
