File: hardware/pcb/receiver/receiver.brd (EAGLE design)
At the start: 100 x 100 mm, 84 parts, among them X1 5-1634506-1H

Commit message: hw/sw: renamed CLKOUT_P/N naming to be the same as in datasheet
Connections:
- net CLKOUT_N renamed CLKOUTB
- net CLKOUT_P renamed CLKOUTA
- net N$48 renamed VCC3P3
- net N$58 renamed VCC_SYS
- removed net N$32: SV1.36
- removed net N$33: SV1.6
- removed net N$35: SV1.38
- removed net N$36: SV1.40
- removed net N$37: SV1.39
- removed net N$38: SV1.37
- removed net N$45: SV1.35
- removed net N$46: SV1.33
- removed net N$52: SV1.5
Changed lines of the file:
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@@
 <?xml version="1.0" encoding="utf-8"?>
 <!DOCTYPE eagle SYSTEM "eagle.dtd">
-<eagle version="7.3.0">
+<eagle version="7.4.0">
 <drawing>
 <settings>
@@
 <signal name="N$57">
 </signal>
-<signal name="CLKOUT_P">
+<signal name="CLKOUTA">
 <contactref element="IC5" pad="41"/>
 <contactref element="SV1" pad="3"/>
@@
 <wire x1="90.62029375" y1="32.82370625" x2="91.44" y2="32.004" width="0.3048" layer="1"/>
 </signal>
-<signal name="CLKOUT_N">
+<signal name="CLKOUTB">
 <contactref element="IC5" pad="40"/>
 <contactref element="SV1" pad="1"/>
@@
 <wire x1="89.84670625" y1="32.32729375" x2="92.71" y2="29.464" width="0.3048" layer="1"/>
 </signal>
-<signal name="N$33">
-<contactref element="SV1" pad="6"/>
-</signal>
-<signal name="N$32">
-<contactref element="SV1" pad="36"/>
-</signal>
-<signal name="N$35">
-<contactref element="SV1" pad="38"/>
-</signal>
-<signal name="N$36">
-<contactref element="SV1" pad="40"/>
-</signal>
-<signal name="N$37">
-<contactref element="SV1" pad="39"/>
-</signal>
-<signal name="N$38">
-<contactref element="SV1" pad="37"/>
-</signal>
-<signal name="N$45">
-<contactref element="SV1" pad="35"/>
-</signal>
-<signal name="N$46">
-<contactref element="SV1" pad="33"/>
-</signal>
-<signal name="N$48">
+<signal name="N$8">
+</signal>
+<signal name="N$21">
+</signal>
+<signal name="VCC3P3">
 <contactref element="SV1" pad="29"/>
 </signal>
-<signal name="N$52">
-<contactref element="SV1" pad="5"/>
-</signal>
-<signal name="N$58">
+<signal name="VCC_SYS">
 <contactref element="SV1" pad="11"/>
 </signal>
-<signal name="N$8">
-</signal>
-<signal name="N$21">
-</signal>
 </signals>
